File: hw/EM-Template.kicad_sch (KiCad schematic)
At the start: 0 parts

Commit message: Changed template to use text variables
Other:
- company: (none) -> Dolvac Instruments
Changed lines of the file:
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@@
-(kicad_sch (version 20230121) (generator eeschema)
-  (paper "A3")
-  (title_block
-    (title "EM-Template")
-    (rev "1.0")
-  )
-  (sheet_instances
-    (path "/" (page "1"))
-  )
+(kicad_sch
+	(version 20250114)
+	(generator "eeschema")
+	(generator_version "9.0")
+	(paper "A3")
+	(title_block
+		(title "EM-Template")
+		(date "${date}")
+		(rev "${rev}")
+		(company "Dolvac Instruments")
+		(comment 1 "SHA: ${sha}")
+	)
+	(sheet_instances
+		(path "/"
+			(page "1")
+		)
+	)
+	(embedded_fonts no)
 )

Commit message: Updated board title card silkscreen
Other:
- title: EM-Template -> ${title}
Changed lines of the file:
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@@
 	(paper "A3")
 	(title_block
-		(title "EM-Template")
+		(title "${title}")
 		(date "${date}")
 		(rev "${rev}")
 		(company "Dolvac Instruments")
 		(comment 1 "SHA: ${sha}")
+		(comment 2 "${desc2}")
+		(comment 3 "${desc1}")
 	)
 	(sheet_instances
